Commit message: test version

File: coco_description/urdf/coco.ros2_control.xacro (robot description, xacro)
@@ -3,5 +3,5 @@
 <ros2_control name="CocoHardware" type="system">
   <hardware>
-    <plugin>pca9685_hardware_interface/Pca9685SystemHardware</plugin>
+    <plugin>coco_hardware/Pca9685SystemHardware</plugin>
   </hardware>
   <joint name="rf_coax_joint">
@@ -53,8 +53,4 @@
     <state_interface name="position"/>
   </joint>
-  <joint name="lb_coax_joint">
-    <command_interface name="position"/>
-    <state_interface name="position"/>
-  </joint>
 </ros2_control>
 </robot>

File: coco_description/urdf/coco.xacro (robot description, xacro)
@@ -2,6 +2,5 @@
 <robot name="coco" xmlns:xacro="http://www.ros.org/wiki/xacro">
 <xacro:include filename="$(find coco_description)/urdf/materials.xacro" />
-<xacro:include filename="$(find coco_description)/urdf/coco.trans" />
-<xacro:include filename="$(find coco_description)/urdf/coco.gazebo" />
+<xacro:include filename="$(find coco_description)/urdf/coco.ros2_control.xacro" />
 <link name="base_link">
   <inertial>
@@ -374,5 +373,5 @@
   <limit upper="0.0" lower="-3.141593" effort="100" velocity="100"/>
 </joint>
-<joint name=" lf_femur_joint" type="revolute">
+<joint name="lf_femur_joint" type="revolute">
   <origin xyz="-0.028498 0.023213 -0.009586" rpy="0 0 0"/>
   <parent link="lf_coax_link_1"/>
