Commit message: working on simulation,all works except controller maneger,changing standar structure

File: coco_description/urdf/coco.gazebo.xacro (robot description, xacro)
@@ -2,5 +2,4 @@
 <robot name="coco" xmlns:xacro="http://www.ros.org/wiki/xacro">
   <!-- Materiales -->
-  <xacro:include filename="$(find coco_description)/urdf/materials.xacro" />
   <!-- Modelo principal (estructura, links, joints) -->
   <xacro:include filename="$(find coco_description)/urdf/coco.xacro" />
@@ -8,5 +7,5 @@
   <ros2_control name="GazeboSystem" type="system">
     <hardware>
-      <plugin>gazebo_ros2_control/GazeboSystem</plugin>
+      <plugin>gz_ros2_control::GazeboSimROS2ControlPlugin/GazeboSystem</plugin>
     </hardware>
     <joint name="rf_coax_joint">
@@ -61,5 +60,7 @@
   <!-- Plugin de Gazebo para ros2_control -->
   <gazebo>
-    <plugin name="gazebo_ros2_control" filename="libgazebo_ros2_control.so"/>
+    <plugin name="gz_ros2_control::GazeboSimROS2ControlPlugin" filename="libgz_ros2_control-system.so">
+        <parameters>/home/justo/Escritorio/Workspaces/coco_ws/src/coco_bringup/config/controllers.yaml </parameters>
+    </plugin>
   </gazebo>
 </robot>

File: coco_description/urdf/coco.xacro (robot description, xacro)
@@ -12,5 +12,5 @@
     <origin xyz="0 0 0" rpy="0 0 0"/>
     <geometry>
-      <mesh filename="package://coco_description/meshes/base_link.stl" scale="0.001 0.001 0.001"/>
+      <mesh filename="file://$(find coco_description)/meshes/base_link.stl" scale="0.001 0.001 0.001"/>
     </geometry>
     <material name="silver"/>
@@ -19,5 +19,5 @@
     <origin xyz="0 0 0" rpy="0 0 0"/>
     <geometry>
-      <mesh filename="package://coco_description/meshes/base_link.stl" scale="0.001 0.001 0.001"/>
+      <mesh filename="file://$(find coco_description)/meshes/base_link.stl" scale="0.001 0.001 0.001"/>
     </geometry>
   </collision>
@@ -32,5 +32,5 @@
     <origin xyz="0.106086 0.004256 0.004897" rpy="0 0 0"/>
     <geometry>
-      <mesh filename="package://coco_description/meshes/rear_link_1.stl" scale="0.001 0.001 0.001"/>
+      <mesh filename="file://$(find coco_description)/meshes/rear_link_1.stl" scale="0.001 0.001 0.001"/>
     </geometry>
     <material name="silver"/>
@@ -39,5 +39,5 @@
     <origin xyz="0.106086 0.004256 0.004897" rpy="0 0 0"/>
     <geometry>
-      <mesh filename="package://coco_description/meshes/rear_link_1.stl" scale="0.001 0.001 0.001"/>
+      <mesh filename="file://$(find coco_description)/meshes/rear_link_1.stl" scale="0.001 0.001 0.001"/>
     </geometry>
   </collision>
@@ -52,5 +52,5 @@
     <origin xyz="-0.115911 0.004871 0.005051" rpy="0 0 0"/>
     <geometry>
-      <mesh filename="package://coco_description/meshes/_front_link_1.stl" scale="0.001 0.001 0.001"/>
+      <mesh filename="file://$(find coco_description)/meshes/_front_link_1.stl" scale="0.001 0.001 0.001"/>
     </geometry>
     <material name="silver"/>
@@ -59,5 +59,5 @@
     <origin xyz="-0.115911 0.004871 0.005051" rpy="0 0 0"/>
     <geometry>
-      <mesh filename="package://coco_description/meshes/_front_link_1.stl" scale="0.001 0.001 0.001"/>
+      <mesh filename="file://$(find coco_description)/meshes/_front_link_1.stl" scale="0.001 0.001 0.001"/>
     </geometry>
   </collision>
@@ -72,5 +72,5 @@
     <origin xyz="0.025005 0.004393 0.060788" rpy="0 0 0"/>
     <geometry>
-      <mesh filename="package://coco_description/meshes/laser_link_1.stl" scale="0.001 0.001 0.001"/>
+      <mesh filename="file://$(find coco_description)/meshes/laser_link_1.stl" scale="0.001 0.001 0.001"/>
     </geometry>
     <material name="silver"/>
@@ -79,5 +79,5 @@
     <origin xyz="0.025005 0.004393 0.060788" rpy="0 0 0"/>
     <geometry>
-      <mesh filename="package://coco_description/meshes/laser_link_1.stl" scale="0.001 0.001 0.001"/>
+      <mesh filename="file://$(find coco_description)/meshes/laser_link_1.stl" scale="0.001 0.001 0.001"/>
     </geometry>
   </collision>
@@ -92,5 +92,5 @@
     <origin xyz="-0.17289 0.043844 -0.001027" rpy="0 0 0"/>
     <geometry>
-      <mesh filename="package://coco_description/meshes/rf_coax_link_1.stl" scale="0.001 0.001 0.001"/>
+      <mesh filename="file://$(find coco_description)/meshes/rf_coax_link_1.stl" scale="0.001 0.001 0.001"/>
     </geometry>
     <material name="silver"/>
@@ -99,5 +99,5 @@
     <origin xyz="-0.17289 0.043844 -0.001027" rpy="0 0 0"/>
     <geometry>
-      <mesh filename="package://coco_description/meshes/rf_coax_link_1.stl" scale="0.001 0.001 0.001"/>
+      <mesh filename="file://$(find coco_description)/meshes/rf_coax_link_1.stl" scale="0.001 0.001 0.001"/>
     </geometry>
   </collision>
@@ -112,5 +112,5 @@
     <origin xyz="-0.172927 -0.034155 -0.001125" rpy="0 0 0"/>
     <geometry>
-      <mesh filename="package://coco_description/meshes/lf_coax_link_1.stl" scale="0.001 0.001 0.001"/>
+      <mesh filename="file://$(find coco_description)/meshes/lf_coax_link_1.stl" scale="0.001 0.001 0.001"/>
     </geometry>
     <material name="silver"/>
@@ -119,5 +119,5 @@
     <origin xyz="-0.172927 -0.034155 -0.001125" rpy="0 0 0"/>
     <geometry>
-      <mesh filename="package://coco_description/meshes/lf_coax_link_1.stl" scale="0.001 0.001 0.001"/>
+      <mesh filename="file://$(find coco_description)/meshes/lf_coax_link_1.stl" scale="0.001 0.001 0.001"/>
     </geometry>
   </collision>
@@ -132,5 +132,5 @@
     <origin xyz="0.106596 0.043339 -0.001713" rpy="0 0 0"/>
     <geometry>
-      <mesh filename="package://coco_description/meshes/rb_coax_link_1.stl" scale="0.001 0.001 0.001"/>
+      <mesh filename="file://$(find coco_description)/meshes/rb_coax_link_1.stl" scale="0.001 0.001 0.001"/>
     </geometry>
     <material name="silver"/>
@@ -139,5 +139,5 @@
     <origin xyz="0.106596 0.043339 -0.001713" rpy="0 0 0"/>
     <geometry>
-      <mesh filename="package://coco_description/meshes/rb_coax_link_1.stl" scale="0.001 0.001 0.001"/>
+      <mesh filename="file://$(find coco_description)/meshes/rb_coax_link_1.stl" scale="0.001 0.001 0.001"/>
     </geometry>
   </collision>
@@ -152,5 +152,5 @@
     <origin xyz="0.106596 -0.034661 -0.001613" rpy="0 0 0"/>
     <geometry>
-      <mesh filename="package://coco_description/meshes/lb_coax_link_1.stl" scale="0.001 0.001 0.001"/>
+      <mesh filename="file://$(find coco_description)/meshes/lb_coax_link_1.stl" scale="0.001 0.001 0.001"/>
     </geometry>
     <material name="silver"/>
@@ -159,5 +159,5 @@
     <origin xyz="0.106596 -0.034661 -0.001613" rpy="0 0 0"/>
     <geometry>
-      <mesh filename="package://coco_description/meshes/lb_coax_link_1.stl" scale="0.001 0.001 0.001"/>
+      <mesh filename="file://$(find coco_description)/meshes/lb_coax_link_1.stl" scale="0.001 0.001 0.001"/>
     </geometry>
   </collision>
@@ -172,5 +172,5 @@
     <origin xyz="0.1351 -0.057832 0.008048" rpy="0 0 0"/>
     <geometry>
-      <mesh filename="package://coco_description/meshes/lb_femur_link_1.stl" scale="0.001 0.001 0.001"/>
+      <mesh filename="file://$(find coco_description)/meshes/lb_femur_link_1.stl" scale="0.001 0.001 0.001"/>
     </geometry>
     <material name="silver"/>
@@ -179,5 +179,5 @@
     <origin xyz="0.1351 -0.057832 0.008048" rpy="0 0 0"/>
     <geometry>
-      <mesh filename="package://coco_description/meshes/lb_femur_link_1.stl" scale="0.001 0.001 0.001"/>
+      <mesh filename="file://$(find coco_description)/meshes/lb_femur_link_1.stl" scale="0.001 0.001 0.001"/>
     </geometry>
   </collision>
@@ -192,5 +192,5 @@
     <origin xyz="-0.144429 -0.057368 0.008461" rpy="0 0 0"/>
     <geometry>
-      <mesh filename="package://coco_description/meshes/lf_femur_link_1.stl" scale="0.001 0.001 0.001"/>
+      <mesh filename="file://$(find coco_description)/meshes/lf_femur_link_1.stl" scale="0.001 0.001 0.001"/>
     </geometry>
     <material name="silver"/>
@@ -199,5 +199,5 @@
     <origin xyz="-0.144429 -0.057368 0.008461" rpy="0 0 0"/>
     <geometry>
-      <mesh filename="package://coco_description/meshes/lf_femur_link_1.stl" scale="0.001 0.001 0.001"/>
+      <mesh filename="file://$(find coco_description)/meshes/lf_femur_link_1.stl" scale="0.001 0.001 0.001"/>
     </geometry>
   </collision>
@@ -212,5 +212,5 @@
     <origin xyz="-0.144371 0.06713 0.008743" rpy="0 0 0"/>
     <geometry>
-      <mesh filename="package://coco_description/meshes/rf_femur_link_1.stl" scale="0.001 0.001 0.001"/>
+      <mesh filename="file://$(find coco_description)/meshes/rf_femur_link_1.stl" scale="0.001 0.001 0.001"/>
     </geometry>
     <material name="silver"/>
@@ -219,5 +219,5 @@
     <origin xyz="-0.144371 0.06713 0.008743" rpy="0 0 0"/>
     <geometry>
-      <mesh filename="package://coco_description/meshes/rf_femur_link_1.stl" scale="0.001 0.001 0.001"/>
+      <mesh filename="file://$(find coco_description)/meshes/rf_femur_link_1.stl" scale="0.001 0.001 0.001"/>
     </geometry>
   </collision>
@@ -232,5 +232,5 @@
     <origin xyz="0.135108 0.066677 0.007984" rpy="0 0 0"/>
     <geometry>
-      <mesh filename="package://coco_description/meshes/rb_femur_link_1.stl" scale="0.001 0.001 0.001"/>
+      <mesh filename="file://$(find coco_description)/meshes/rb_femur_link_1.stl" scale="0.001 0.001 0.001"/>
     </geometry>
     <material name="silver"/>
@@ -239,5 +239,5 @@
     <origin xyz="0.135108 0.066677 0.007984" rpy="0 0 0"/>
     <geometry>
-      <mesh filename="package://coco_description/meshes/rb_femur_link_1.stl" scale="0.001 0.001 0.001"/>
+      <mesh filename="file://$(find coco_description)/meshes/rb_femur_link_1.stl" scale="0.001 0.001 0.001"/>
     </geometry>
   </collision>
@@ -252,5 +252,5 @@
     <origin xyz="0.242628 -0.063618 0.010796" rpy="0 0 0"/>
     <geometry>
-      <mesh filename="package://coco_description/meshes/lb_tibia_link_1.stl" scale="0.001 0.001 0.001"/>
+      <mesh filename="file://$(find coco_description)/meshes/lb_tibia_link_1.stl" scale="0.001 0.001 0.001"/>
     </geometry>
     <material name="silver"/>
@@ -259,5 +259,5 @@
     <origin xyz="0.242628 -0.063618 0.010796" rpy="0 0 0"/>
     <geometry>
-      <mesh filename="package://coco_description/meshes/lb_tibia_link_1.stl" scale="0.001 0.001 0.001"/>
+      <mesh filename="file://$(find coco_description)/meshes/lb_tibia_link_1.stl" scale="0.001 0.001 0.001"/>
     </geometry>
   </collision>
@@ -272,5 +272,5 @@
     <origin xyz="-0.036894 -0.063154 0.0109" rpy="0 0 0"/>
     <geometry>
-      <mesh filename="package://coco_description/meshes/lf_tibia_link_1.stl" scale="0.001 0.001 0.001"/>
+      <mesh filename="file://$(find coco_description)/meshes/lf_tibia_link_1.stl" scale="0.001 0.001 0.001"/>
     </geometry>
     <material name="silver"/>
@@ -279,5 +279,5 @@
     <origin xyz="-0.036894 -0.063154 0.0109" rpy="0 0 0"/>
     <geometry>
-      <mesh filename="package://coco_description/meshes/lf_tibia_link_1.stl" scale="0.001 0.001 0.001"/>
+      <mesh filename="file://$(find coco_description)/meshes/lf_tibia_link_1.stl" scale="0.001 0.001 0.001"/>
     </geometry>
   </collision>
@@ -292,5 +292,5 @@
     <origin xyz="-0.036961 0.072914 0.011343" rpy="0 0 0"/>
     <geometry>
-      <mesh filename="package://coco_description/meshes/rf_tibia_link_1.stl" scale="0.001 0.001 0.001"/>
+      <mesh filename="file://$(find coco_description)/meshes/rf_tibia_link_1.stl" scale="0.001 0.001 0.001"/>
     </geometry>
     <material name="silver"/>
@@ -299,5 +299,5 @@
     <origin xyz="-0.036961 0.072914 0.011343" rpy="0 0 0"/>
     <geometry>
-      <mesh filename="package://coco_description/meshes/rf_tibia_link_1.stl" scale="0.001 0.001 0.001"/>
+      <mesh filename="file://$(find coco_description)/meshes/rf_tibia_link_1.stl" scale="0.001 0.001 0.001"/>
     </geometry>
   </collision>
@@ -312,5 +312,5 @@
     <origin xyz="0.242508 0.072461 0.010989" rpy="0 0 0"/>
     <geometry>
-      <mesh filename="package://coco_description/meshes/rb_tibia_link_1.stl" scale="0.001 0.001 0.001"/>
+      <mesh filename="file://$(find coco_description)/meshes/rb_tibia_link_1.stl" scale="0.001 0.001 0.001"/>
     </geometry>
     <material name="silver"/>
@@ -319,5 +319,5 @@
     <origin xyz="0.242508 0.072461 0.010989" rpy="0 0 0"/>
     <geometry>
-      <mesh filename="package://coco_description/meshes/rb_tibia_link_1.stl" scale="0.001 0.001 0.001"/>
+      <mesh filename="file://$(find coco_description)/meshes/rb_tibia_link_1.stl" scale="0.001 0.001 0.001"/>
     </geometry>
   </collision>
