Commit message: renamed joints

File: coco_description/urdf/coco.xacro (robot description, xacro)
@@ -246,5 +246,5 @@
 <link name="lb_tibia_link_1">
   <inertial>
-    <origin xyz="-0.03196384904823907 0.02772555624743414 0.0038597457608928057" rpy="0 0 0"/>
+    <origin xyz="-0.03196384904823907 0.027725556247434155 0.003859745760892816" rpy="0 0 0"/>
     <mass value="0.10314122455204974"/>
     <inertia ixx="1.8e-05" iyy="0.000196" izz="0.0002" ixy="-0.0" iyz="-1e-06" ixz="1.3e-05"/>
@@ -266,5 +266,5 @@
 <link name="lf_tibia_link_1">
   <inertial>
-    <origin xyz="-0.03197671433292928 0.02772553703112078 0.0037573349954613177" rpy="0 0 0"/>
+    <origin xyz="-0.031976714332929285 0.02772553703112078 0.0037573349954613177" rpy="0 0 0"/>
     <mass value="0.10314122455337109"/>
     <inertia ixx="1.8e-05" iyy="0.000196" izz="0.0002" ixy="-0.0" iyz="-1e-06" ixz="1.3e-05"/>
@@ -286,5 +286,5 @@
 <link name="rf_tibia_link_1">
   <inertial>
-    <origin xyz="-0.031502492319461874 -0.027791020823839455 0.0062624864037398" rpy="0 0 0"/>
+    <origin xyz="-0.031502492319461874 -0.02779102082383947 0.0062624864037398" rpy="0 0 0"/>
     <mass value="0.10311453435844117"/>
     <inertia ixx="2.1e-05" iyy="0.000196" izz="0.000197" ixy="-0.0" iyz="1e-06" ixz="2.7e-05"/>
@@ -374,5 +374,5 @@
   <limit upper="0.0" lower="-3.141593" effort="100" velocity="100"/>
 </joint>
-<joint name="Revoluci�n 10" type="revolute">
+<joint name=" lf_femur_joint" type="revolute">
   <origin xyz="-0.028498 0.023213 -0.009586" rpy="0 0 0"/>
   <parent link="lf_coax_link_1"/>
@@ -381,5 +381,5 @@
   <limit upper="0.0" lower="-3.141593" effort="100" velocity="100"/>
 </joint>
-<joint name="Revoluci�n 11" type="revolute">
+<joint name="rf_femur_joint" type="revolute">
   <origin xyz="-0.028519 -0.023286 -0.00977" rpy="0 0 0"/>
   <parent link="rf_coax_link_1"/>
@@ -388,5 +388,5 @@
   <limit upper="3.141593" lower="0.0" effort="100" velocity="100"/>
 </joint>
-<joint name="Revoluci�n 12" type="revolute">
+<joint name="rb_femur_joint" type="revolute">
   <origin xyz="-0.028512 -0.023338 -0.009697" rpy="0 0 0"/>
   <parent link="rb_coax_link_1"/>
@@ -395,5 +395,5 @@
   <limit upper="3.141593" lower="0.0" effort="100" velocity="100"/>
 </joint>
-<joint name="Revoluci�n 13" type="revolute">
+<joint name="lb_tibia_joint" type="revolute">
   <origin xyz="-0.107528 0.005786 -0.002748" rpy="0 0 0"/>
   <parent link="lb_femur_link_1"/>
@@ -402,5 +402,5 @@
   <limit upper="0.0" lower="-2.617994" effort="100" velocity="100"/>
 </joint>
-<joint name="Revoluci�n 14" type="revolute">
+<joint name="lf_tibia_joint" type="revolute">
   <origin xyz="-0.107535 0.005786 -0.002439" rpy="0 0 0"/>
   <parent link="lf_femur_link_1"/>
@@ -409,5 +409,5 @@
   <limit upper="0.0" lower="-2.617994" effort="100" velocity="100"/>
 </joint>
-<joint name="Revoluci�n 15" type="revolute">
+<joint name="rf_tibia_joint" type="revolute">
   <origin xyz="-0.10741 -0.005784 -0.0026" rpy="0 0 0"/>
   <parent link="rf_femur_link_1"/>
@@ -416,5 +416,5 @@
   <limit upper="2.617994" lower="0.0" effort="100" velocity="100"/>
 </joint>
-<joint name="Revoluci�n 16" type="revolute">
+<joint name="rb_tibia_joint" type="revolute">
   <origin xyz="-0.1074 -0.005784 -0.003005" rpy="0 0 0"/>
   <parent link="rb_femur_link_1"/>

Commit message: adding lidar

File: coco_description/urdf/coco.xacro (robot description, xacro)
@@ -63,5 +63,5 @@
   </collision>
 </link>
-<link name="laser_link_1">
+<link name="laser">
   <inertial>
     <origin xyz="8.838579649582401e-06 -0.0005477770066574924 -0.017396902560964038" rpy="0 0 0"/>
@@ -334,7 +334,7 @@
 </joint>
 <joint name="base_link_to_lidar_joint" type="fixed">
-  <origin xyz="-0.025005 -0.004393 -0.060788" rpy="0 0 0"/>
+  <origin xyz="-0.025005 -0.004393 -0.060788" rpy="3.14159 0 3.14159"/>
   <parent link="base_link"/>
-  <child link="laser_link_1"/>
+  <child link="laser"/>
 </joint>
 <joint name="rf_coax_joint" type="revolute">

Commit message: integrating imu and lidar fusion

File: coco_description/urdf/coco.xacro (robot description, xacro)
@@ -23,4 +23,24 @@
   </collision>
 </link>
+<link name="imu_link">
+  <inertial>
+    <origin xyz="-0.1171941 -0.01 -0.0302" rpy="0 0 1.57"/>
+    <mass value="0.01"/>
+    <inertia
+      ixx="1e-6" iyy="1e-6" izz="1e-6"
+      ixy="0" ixz="0" iyz="0"/>
+  </inertial>
+  <visual>
+    <origin xyz="0 0 0" rpy="0 0 0"/>
+    <geometry><box size="0.02 0.02 0.02"/></geometry>
+    <material name="Blue"/>
+  </visual>
+</link>
+<joint name="base_to_imu" type="fixed">
+  <!-- 10 cm hacia atrás en X -->
+  <origin xyz="-0.10 0 0" rpy="0 0 0"/>
+  <parent link="base_link"/>
+  <child  link="imu_link"/>
+</joint>
 <link name="rear_link_1">
   <inertial>

Commit message: Added odom frame

File: coco_description/urdf/coco.xacro (robot description, xacro)
@@ -3,4 +3,10 @@
 <xacro:include filename="$(find coco_description)/urdf/materials.xacro" />
 <xacro:include filename="$(find coco_description)/urdf/coco.ros2_control.xacro" />
+<link name="odom"/>
+  <joint name="odom_to_base" type="fixed">
+    <parent link="odom"/>
+    <child  link="base_link"/>
+    <origin xyz="0 0 0" rpy="0 0 0"/>
+  </joint>
 <link name="base_link">
   <inertial>
@@ -25,5 +31,5 @@
 <link name="imu_link">
   <inertial>
-    <origin xyz="-0.1171941 -0.01 -0.0302" rpy="0 0 1.57"/>
+    <origin xyz="-0.0171941 -0.01 -0.0302" rpy="0 0 0"/>
     <mass value="0.01"/>
     <inertia
@@ -34,10 +40,9 @@
     <origin xyz="0 0 0" rpy="0 0 0"/>
     <geometry><box size="0.02 0.02 0.02"/></geometry>
-    <material name="Blue"/>
+    <material name="silver"/>
   </visual>
 </link>
 <joint name="base_to_imu" type="fixed">
-  <!-- 10 cm hacia atrás en X -->
-  <origin xyz="-0.10 0 0" rpy="0 0 0"/>
+  <origin xyz="0.0 0 0" rpy="0 0 0"/>
   <parent link="base_link"/>
   <child  link="imu_link"/>

Commit message: added map, odom and base_footprint and nav2 params file

File: coco_description/urdf/coco.xacro (robot description, xacro)
@@ -3,10 +3,12 @@
 <xacro:include filename="$(find coco_description)/urdf/materials.xacro" />
 <xacro:include filename="$(find coco_description)/urdf/coco.ros2_control.xacro" />
+<link name="map"/>
 <link name="odom"/>
-  <joint name="odom_to_base" type="fixed">
-    <parent link="odom"/>
-    <child  link="base_link"/>
-    <origin xyz="0 0 0" rpy="0 0 0"/>
-  </joint>
+<link name="base_footprint"/>
+<joint name="odom_to_footprint" type="fixed">
+  <parent link="odom"/>
+  <child  link="base_footprint"/>
+  <origin xyz="0 0 0" rpy="0 0 0"/>
+</joint>
 <link name="base_link">
   <inertial>
@@ -29,4 +31,10 @@
   </collision>
 </link>
+<joint name="footprint_to_base" type="fixed">
+  <parent link="base_footprint"/>
+  <child  link="base_link"/>
+  <!-- set at standby high -->
+  <origin xyz="0 0 0.2" rpy="0 0 0"/>
+</joint>
 <link name="imu_link">
   <inertial>

Commit message: fixed error in urdf

File: coco_description/urdf/coco.xacro (robot description, xacro)
@@ -3,12 +3,5 @@
 <xacro:include filename="$(find coco_description)/urdf/materials.xacro" />
 <xacro:include filename="$(find coco_description)/urdf/coco.ros2_control.xacro" />
-<link name="map"/>
-<link name="odom"/>
 <link name="base_footprint"/>
-<joint name="odom_to_footprint" type="fixed">
-  <parent link="odom"/>
-  <child  link="base_footprint"/>
-  <origin xyz="0 0 0" rpy="0 0 0"/>
-</joint>
 <link name="base_link">
   <inertial>
